Commit message: Jacobian-wip

File: Project/urdf/SC_2DoF.urdf (robot description, URDF)
Before this commit: robot Chaser, 4 links, 3 joints
Links:
- removed link Link_1
- removed link Link_2
- removed link Link_EE
- added link Link1, mass 5; visual cylinder length=0.1 radius=0.1; visual cylinder length=1 radius=0.05
- added link Link2, mass 2.5; visual cylinder length=0.15 radius=0.075; visual cylinder length=0.5 radius=0.05
- added link endeffector, mass 0; visual sphere radius=0.1
- link Spacecraft: mass 100 -> 10
Joints:
- removed joint Joint_1
- removed joint Joint_2
- removed joint Joint_EE
- added joint jnt1: type revolute, parent Spacecraft, child Link1, origin xyz=0.5 0 0 rpy=0 0 0, axis 0 0 1, limit effort=0 velocity=0
- added joint jnt2: type revolute, parent Link1, child Link2, origin xyz=1 0 0 rpy=0 0 0, axis 0 0 1, limit effort=0 velocity=0
- added joint jnt_ee: type fixed, parent Link2, child endeffector, origin xyz=0.5 0 0 rpy=0 0 0, axis 1 0 0
