Commit message: New mats to bodies
R, A, P, M

File: Project/urdf/ModelTest.urdf (robot description, URDF)
Before this commit: robot Chaser, 4 links, 3 joints
Links:
- removed link Link1
- removed link Link2
- removed link Spacecraft
- removed link endeffector
Joints:
- joint jnt1: child Link1 -> ; parent Spacecraft -> 
- joint jnt2: child Link2 -> ; parent Link1 -> 
- joint jntEE: child endeffector -> ; parent Link2 -> 

File: Project/urdf/SC_2DoF.urdf (robot description, URDF)
Before this commit: robot Chaser, 4 links, 3 joints
Links:
- removed link Link1
- removed link Link2
- removed link Spacecraft
- removed link endeffector
Joints:
- joint jnt1: child Link1 -> ; parent Spacecraft -> 
- joint jnt2: child Link2 -> ; parent Link1 -> 
- joint jnt_ee: child endeffector -> ; parent Link2 -> 

File: Project/urdf/SC_3DoF_old.urdf (robot description, URDF)
Before this commit: robot Chaser, 6 links, 5 joints
Links:
- removed link Link_0
- removed link Link_1
- removed link Link_2
- removed link Link_3
- removed link Link_EE
- removed link Spacecraft
Joints:
- joint Joint_1: child Link_1 -> ; parent Link_0 -> 
- joint Joint_2: child Link_2 -> ; parent Link_1 -> 
- joint Joint_3: child Link_3 -> ; parent Link_2 -> 
- joint Joint_EE: child Link_EE -> ; parent Link_3 -> 
- joint Spacecraft_Manipulator_Joint: child Link_0 -> ; parent Spacecraft -> 

File: Project/urdf/SC_3Link.urdf (robot description, URDF)
Before this commit: robot Chaser, 6 links, 5 joints
Links:
- removed link Link_0
- removed link Link_1
- removed link Link_2
- removed link Link_3
- removed link Link_EE
- removed link Spacecraft
Joints:
- joint Joint_1: child Link_1 -> ; parent Link_0 -> 
- joint Joint_2: child Link_2 -> ; parent Link_1 -> 
- joint Joint_3: child Link_3 -> ; parent Link_2 -> 
- joint Joint_EE: child Link_EE -> ; parent Link_3 -> 
- joint Spacecraft_Manipulator_Joint: child Link_0 -> ; parent Spacecraft -> 

Commit message: fixed urdf

File: Project/urdf/ModelTest.urdf (robot description, URDF)
Before this commit: robot Chaser, 0 links, 3 joints
Links:
- added link Link1, mass 5; visual cylinder length=0.1 radius=0.1; visual cylinder length=1 radius=0.05
- added link Link2, mass 5; visual cylinder length=0.15 radius=0.075; visual cylinder length=0.5 radius=0.05
- added link Spacecraft, mass 100; visual box size=0.25 0.25 0.25
- added link endeffector, mass 0; visual sphere radius=0.1
Joints:
- joint jnt1: child  -> Link1; parent  -> Spacecraft
- joint jnt2: child  -> Link2; parent  -> Link1
- joint jntEE: child  -> endeffector; parent  -> Link2

File: Project/urdf/SC_2DoF.urdf (robot description, URDF)
Before this commit: robot Chaser, 0 links, 3 joints
Links:
- added link Link1, mass 5; visual cylinder length=0.1 radius=0.1; visual cylinder length=1 radius=0.05
- added link Link2, mass 2.5; visual cylinder length=0.15 radius=0.075; visual cylinder length=0.5 radius=0.05
- added link Spacecraft, mass 10; visual box size=1 1 1
- added link endeffector, mass 0; visual sphere radius=0.1
Joints:
- joint jnt1: child  -> Link1; parent  -> Spacecraft
- joint jnt2: child  -> Link2; parent  -> Link1
- joint jnt_ee: child  -> endeffector; parent  -> Link2

File: Project/urdf/SC_3DoF_old.urdf (robot description, URDF)
Before this commit: robot Chaser, 0 links, 5 joints
Links:
- added link Link_0, mass 5; visual cylinder length=0.25 radius=0.05
- added link Link_1, mass 5; visual cylinder length=0.1 radius=0.1; visual cylinder length=0.2 radius=0.05
- added link Link_2, mass 10; visual cylinder length=0.15 radius=0.075; visual cylinder length=0.75 radius=0.05
- added link Link_3, mass 10; visual cylinder length=0.15 radius=0.075; visual cylinder length=2 radius=0.05
- added link Link_EE, mass 0; visual sphere radius=0.1
- added link Spacecraft, mass 100; visual box size=0.75 0.75 0.75
Joints:
- joint Joint_1: child  -> Link_1; parent  -> Link_0
- joint Joint_2: child  -> Link_2; parent  -> Link_1
- joint Joint_3: child  -> Link_3; parent  -> Link_2
- joint Joint_EE: child  -> Link_EE; parent  -> Link_3
- joint Spacecraft_Manipulator_Joint: child  -> Link_0; parent  -> Spacecraft

File: Project/urdf/SC_3Link.urdf (robot description, URDF)
Before this commit: robot Chaser, 0 links, 5 joints
Links:
- added link Link_0, mass 1; visual cylinder length=0.25 radius=0.05
- added link Link_1, mass 10; visual cylinder length=0.1 radius=0.1; visual cylinder length=2 radius=0.05
- added link Link_2, mass 10; visual cylinder length=0.15 radius=0.075; visual cylinder length=2 radius=0.05
- added link Link_3, mass 10; visual cylinder length=0.15 radius=0.075; visual cylinder length=2 radius=0.05
- added link Link_EE, mass 0; visual sphere radius=0.1
- added link Spacecraft, mass 100; visual box size=2.5 2.5 2.5
Joints:
- joint Joint_1: child  -> Link_1; parent  -> Link_0
- joint Joint_2: child  -> Link_2; parent  -> Link_1
- joint Joint_3: child  -> Link_3; parent  -> Link_2
- joint Joint_EE: child  -> Link_EE; parent  -> Link_3
- joint Spacecraft_Manipulator_Joint: child  -> Link_0; parent  -> Spacecraft
